File: keyboard-template-60.kicad_pcb (KiCad board)
At the start: 2 copper layers, 171 parts, among them J1 USB_C_Receptacle_USB2.0, J2 Conn_01x04_MountingPin, SW1 SW_Reset, U1 ATmega32U4-A, U2 SRV05-4, Y1 16MHz

Commit message: Place PCB outline and parts
Parts:
- added REF**: 60_Outline, locallib:60_Outline-Modded, F.Cu at (206.4, 127.0)
- C1, C2, C3, C4, C5, C6, C7, C8, D1, D10, D11, D12, D13, D14, D15, D16, D17, D18, D19, D2, D20, D21, D22, D24, D25, D26, D27, D28, D29, D3, D30, D31, D32, D33, D34, D35, D36, D37, D39, D4, D40, D41, D42, D43, D44, D45, D46, D47, D48, D49, D5, D50, D51, D52, D53, D54, D55, D56, D57, D58, D59, D6, D60, D61, D62, D63, D64, D65, D67, D68, D69, D7, D71, D72, D73, D74, D75, D8, D9, F1, J1, J2, MX1, MX10, MX11, MX12, MX13, MX14, MX15, MX16, MX17, MX18, MX19, MX2, MX20, MX21, MX22, MX24, MX25, MX26, MX27, MX28, MX29, MX3, MX30, MX39, MX39-2, MX4, MX40, MX41, MX42, MX43, MX44, MX45, MX46, MX47, MX48, MX49, MX5, MX50, MX51, MX52, MX53, MX54, MX55, MX56, MX57, MX58, MX59, MX6, MX60, MX61, MX62, MX63, MX63-2, MX64, MX64-2, MX65, MX65-2, MX67, MX68, MX69, MX7, MX71, MX71-2, MX72, MX72-2, MX73, MX73-2, MX74, MX75, MX8, MX9, R1, R2, R3, R4, R5, R6, SW1, U1, U2, Y1: moved to B.Cu
- MX31: renamed from MX32; moved to B.Cu
- MX32: renamed from MX33; moved to B.Cu
- MX33: renamed from MX34; moved to B.Cu
- MX34: renamed from MX35; moved to B.Cu
- MX35: renamed from MX36; moved to B.Cu
- MX36: renamed from MX37; moved to B.Cu
- MX37: renamed from MX38; moved to B.Cu
- MX37-2: renamed from MX38-2; moved to B.Cu
- moved MX63 571.2 mm to (582.6, 411.2), turned to 180 degrees
- moved MX46 569.4 mm to (620.7, 392.1), turned to 180 degrees
- moved MX2 548.6 mm to (601.7, 335.0), turned to 180 degrees
- moved MX1 542.7 mm to (620.7, 335.0), turned to 180 degrees
- moved MX16 535.5 mm to (611.2, 354.0), turned to 180 degrees
- moved MX65 528.8 mm to (544.5, 411.2), turned to 180 degrees
- moved MX33 524.7 mm to (577.9, 373.1), turned to 180 degrees
- moved MX34 523.9 mm to (558.8, 373.1), turned to 180 degrees
- moved MX19 518.8 mm to (554.0, 354.0), turned to 180 degrees
- moved MX49 507.9 mm to (563.6, 392.1), turned to 180 degrees
- moved MX61 499.6 mm to (620.7, 411.2), turned to 180 degrees
- moved MX20 496.8 mm to (535.0, 354.0), turned to 180 degrees
- moved MX17 494.7 mm to (592.1, 354.0), turned to 180 degrees
- moved MX62 493.9 mm to (601.7, 411.2), turned to 180 degrees
- moved MX37-2 490.4 mm to (499.3, 373.1)
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Other:
- board outline added: 285 x 95.1 mm

Commit message: Continue placing parts
Parts:
- MX16, MX30: footprint marbastlib-mx:SW_MX_HS_1u -> marbastlib-mx:SW_MX_HS_1.5u
- MX31, MX37-2, MX39-2, MX45: footprint marbastlib-mx:SW_MX_HS_1u -> marbastlib-mx:SW_MX_HS_1.25u
- MX67, MX69: footprint marbastlib-mx:SW_MX_HS_1u -> MX_Only:MXOnly-2U-Hotswap-ReversedStabilizers; moved to F.Cu
- MX68: footprint marbastlib-mx:SW_MX_HS_1u -> MX_Only:MXOnly-7U-Hotswap-ReversedStabilizers; moved to F.Cu
- moved MX30 377.1 mm to (77.8, 108.0)
- moved MX45 375.3 mm to (75.4, 127.0)
- moved MX17 373.5 mm to (311.1, 108.0)
- moved MX36 373.5 mm to (239.7, 127.0)
- moved MX50 373.5 mm to (263.5, 146.1)
- moved MX65 373.5 mm to (263.5, 165.1)
- moved MX5 373.5 mm to (263.5, 88.9)
- moved MX12 373.5 mm to (130.2, 88.9)
- moved MX13 373.5 mm to (111.1, 88.9)
- moved MX14 373.5 mm to (92.1, 88.9)
- moved MX19 373.5 mm to (273.1, 108.0)
- moved MX2 373.5 mm to (320.7, 88.9)
- moved MX21 373.5 mm to (234.9, 108.0)
- moved MX25 373.5 mm to (177.8, 108.0)
- moved MX26 373.5 mm to (158.8, 108.0)
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
Commit message: Continue placing parts
Parts:
- moved D13 479.8 mm to (165.1, 42.1)
- moved D3 461.5 mm to (228.6, 42.1)
- moved D43 458.8 mm to (165.1, 54.8)
- moved D9 457.2 mm to (190.5, 42.1)
- moved D27 456.3 mm to (171.4, 48.4)
- moved D19 454.3 mm to (222.2, 48.4)
- moved D1 454.2 mm to (241.3, 42.1)
- moved D41 453.9 mm to (177.8, 54.8)
- moved D34 452.9 mm to (222.2, 54.8)
- moved D25 452.9 mm to (184.2, 48.4)
- moved D32 451.3 mm to (234.9, 54.8)
- moved D31 451.2 mm to (241.3, 54.8)
- moved D36 441.8 mm to (209.6, 54.8)
- moved D26 430.8 mm to (177.8, 48.4)
- moved D15 414.2 mm to (152.4, 42.1)
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
Commit message: Update the schematic and fix the order of footprints on the PCB
Parts:
- added S1: MX_stab, marbastlib-mx:STAB_MX_2u, F.Cu at (173.8, 217.5)
- added S2: MX_stab, marbastlib-mx:STAB_MX_2u, F.Cu at (218.3, 219.9)
- added S3: MX_stab, marbastlib-mx:STAB_MX_7u, F.Cu at (206.4, 165.1)
- MX67, MX69: footprint MX_Only:MXOnly-2U-Hotswap-ReversedStabilizers -> marbastlib-mx:SW_MX_HS_1u; moved to B.Cu
- MX68: footprint MX_Only:MXOnly-7U-Hotswap-ReversedStabilizers -> marbastlib-mx:SW_MX_HS_1u; moved to B.Cu
- moved MX1 266.7 mm to (73.0, 88.9)
- moved MX15 266.7 mm to (339.7, 88.9)
- moved MX31 264.8 mm to (84.9, 46.8)
- moved MX16 257.2 mm to (77.8, 108.0)
- moved MX30 257.2 mm to (335.0, 108.0)
- moved MX14 228.6 mm to (320.7, 88.9)
- moved MX2 228.6 mm to (92.1, 88.9)
- moved MX32 224.4 mm to (106.4, 46.8)
- moved MX17 209.5 mm to (101.6, 108.0)
- moved MX29 209.5 mm to (311.1, 108.0)
- moved MX13 190.5 mm to (301.6, 88.9)
- moved MX3 190.5 mm to (111.1, 88.9)
- moved MX18 171.5 mm to (120.7, 108.0)
- moved MX28 171.5 mm to (292.1, 108.0)
- moved MX12 152.4 mm to (282.6, 88.9)
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
Commit message: Update the gs
Parts:
- moved MX46 266.7 mm to (73.0, 146.1)
- moved MX60 266.7 mm to (339.7, 146.1)
- moved MX61 266.7 mm to (73.0, 165.1)
- moved MX75 266.7 mm to (339.7, 165.1)
- moved MX45 261.9 mm to (337.3, 127.0)
- moved MX47 228.6 mm to (92.1, 146.1)
- moved MX59 228.6 mm to (320.7, 146.1)
- moved MX62 228.6 mm to (92.1, 165.1)
- moved MX74 228.6 mm to (320.7, 165.1)
- moved MX44 219.1 mm to (315.9, 127.0)
- moved MX48 190.5 mm to (111.1, 146.1)
- moved MX58 190.5 mm to (301.6, 146.1)
- moved MX63 190.5 mm to (111.1, 165.1)
- moved MX73 190.5 mm to (301.6, 165.1)
- moved MX33 181.0 mm to (115.9, 127.0)
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