File: keyboard-template-60.kicad_pcb (KiCad board)
At the start: 2 copper layers, 285 x 95.1 mm, 169 parts, among them J1 USB_C_Receptacle_USB2.0, J2 Conn_01x04_MountingPin, SW1 SW_Reset, U1 ATmega32U4-A, U2 SRV05-4, Y1 16MHz

Commit message: Update MCU footprint GND new
Connections:
- U1 pad 45: (no net) -> GND
Routing:
- net GND: track 104.7 -> 73.0 mm, vias 6 -> 0

Commit message: Gerbers
Parts:
- U1: value ATmega32U4-A -> ATmega32U4-M
Routing:
- net GND: track 73.0 -> 125.2 mm, vias 0 -> 6
- net ROW0: track 329.0 -> 329.8 mm

Commit message: Update schematics and BOM
Parts:
- moved D46 0.79 mm to (86.5, 150.8)
Connections:
- U1 pad 11: unconnected-(U1-Pad11) -> COL1
- U1 pad 38: COL1 -> ROW4
- U1 pad 39: ROW4 -> unconnected-(U1-Pad39)
Routing:
- net COL1: track 160.5 -> 126.1 mm, vias 0 -> 1
- net ROW4: track 340.0 -> 334.4 mm
- net COL6: track 241.8 -> 242.5 mm
- net COL2: track 146.0 -> 146.7 mm

Commit message: Updates to the PCB layout
Parts:
- moved D45 18.3 mm to (327.0, 127.0)
- moved D37 5.56 mm to (204.8, 127.0)
- moved D39 5.56 mm to (208.0, 127.0)
- moved D15 4.63 mm to (342.9, 94.5)
- moved D60 3.97 mm to (342.9, 152.4)
- moved D75 2.38 mm to (342.9, 169.1)
- moved R4 0.79 mm to (89.7, 84.9)
- turned MX39 to 0 degrees
- turned MX39-2 to 180 degrees
Routing:
- net GND: track 125.2 -> 75.5 mm, vias 6 -> 0
- net ROW2: track 301.7 -> 277.6 mm
- net COL8: track 276.3 -> 287.5 mm
- net Net-(D45-Pad2): track 4.20 -> 14.7 mm
- net ROW1: track 278.4 -> 288.4 mm
- net COL6: track 242.5 -> 248.8 mm
- net 39-2: track 35.8 -> 41.1 mm
- net ROW0: track 329.8 -> 334.7 mm
- net COL10: track 285.5 -> 289.7 mm
- net COL7: track 220.2 -> 224.4 mm
- net COL2: track 146.7 -> 150.9 mm
- net Net-(D15-Pad2): track 13.4 -> 9.25 mm
- net ROW3: track 312.0 -> 308.0 mm
- net Net-(D60-Pad2): track 13.4 -> 10.0 mm
- net unconnected-(J2-PadMP): track 8.41 -> 5.60 mm, vias 2 -> 0
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Other:
- board size 285 x 95.1 mm -> 285 x 94.6 mm
